File: TKL 40.kicad_pcb (KiCad board)
At the start: 2 copper layers, 122 parts, among them SW1 SW_Push, SW10 SW_Push, SW11 SW_Push, SW12 SW_Push, SW13 SW_Push, SW14 SW_Push, SW15 SW_Push, SW16 SW_Push, SW17 SW_Push, SW18 SW_Push, SW19 SW_Push, SW2 SW_Push, SW20 SW_Push, SW21 SW_Push, SW22 SW_Push, SW23 SW_Push, SW24 SW_Push, SW24_1 SW_Push, SW25 SW_Push, SW26 SW_Push, SW27 SW_Push, SW28 SW_Push, SW29 SW_Push, SW3 SW_Push, SW30 SW_Push, SW31 SW_Push, SW32 SW_Push, SW33 SW_Push, SW34 SW_Push, SW35 SW_Push, SW35_1 SW_Push, SW35_2 SW_Push, SW36 SW_Push, SW36_1 SW_Push, SW37 SW_Push, SW38 SW_Push, SW39 SW_Push, SW4 SW_Push, SW40 SW_Push, SW41 SW_Push, SW42 SW_Push, SW43 SW_Push, SW44 SW_Push, SW45 SW_Push, SW46 SW_Push, SW47 SW_Push, SW47_1 SW_Push, SW48 SW_Push, SW48_1 SW_Push, SW49 SW_Push, SW5 SW_Push, SW50 SW_Push, SW51 SW_Push, SW52 SW_Push, SW53 SW_Push, SW54 SW_Push, SW55 SW_Push, SW56 SW_Push, SW56_1 SW_Push, SW57 SW_Push, SW57_1 SW_Push, SW6 SW_Push, SW7 SW_Push, SW8 SW_Push, SW9 SW_Push

Commit message: Added MCU, ESD, and some routing
Parts:
- added BOOT: RST, Button_Switch_SMD:SW_SPST_SKQG_WithoutStem, B.Cu at (194.8, 114.0)
- added C1: 100nF, Capacitor_SMD:C_0402_1005Metric, B.Cu at (188.8, 121.0)
- added C2: 4.7uF, Capacitor_SMD:C_0402_1005Metric, B.Cu at (113.5, 108.5)
- added C3: 100nF, Capacitor_SMD:C_0402_1005Metric, B.Cu at (110.2, 122.5)
- added C4: 100nF, Capacitor_SMD:C_0402_1005Metric, B.Cu at (108.5, 110.5)
- added C5: 100nF, Capacitor_SMD:C_0402_1005Metric, B.Cu at (107.8, 120.0)
- added C6: 100nF, Capacitor_SMD:C_0402_1005Metric, B.Cu at (120.0, 113.5)
- added C7: 100nF, Capacitor_SMD:C_0402_1005Metric, B.Cu at (116.5, 122.8)
- added C8: 1uF, Capacitor_SMD:C_0402_1005Metric, B.Cu at (120.3, 68.5)
- added C9: 1uF, Capacitor_SMD:C_0402_1005Metric, B.Cu at (118.0, 70.9)
- added J1: JST, acheron_Connectors.pretty-master:MOLEX_781710004_MountingReliefs, B.Cu at (125.8, 50.4)
- added R1: 10k, Resistor_SMD:R_0402_1005Metric, B.Cu at (188.8, 117.5)
- added RESET: RST, Button_Switch_SMD:SW_SPST_SKQG_WithoutStem, B.Cu at (194.8, 121.2)
- added U1: STM32F072C8Tx, Package_QFP:LQFP-48_7x7mm_P0.5mm, B.Cu at (113.2, 116.0)
- added U2: XC6206PxxxMR-Regulator_Linear, Package_TO_SOT_SMD:SOT-23, B.Cu at (118.0, 68.5)
Routing:
- net COL11: track 184.4 -> 350.0 mm
- net +3V3: track 0.00 -> 159.7 mm, vias 0 -> 7
- net GND: track 0.00 -> 128.5 mm, vias 0 -> 3
- net COL10: track 129.9 -> 242.4 mm
- net NRST: track 0.00 -> 101.2 mm, vias 0 -> 2
- net COL9: track 99.9 -> 192.6 mm
- net BOOT0: track 0.00 -> 89.7 mm
- net COL8: track 77.5 -> 164.7 mm, vias 0 -> 2
- net ROW1: track 208.0 -> 293.7 mm, vias 0 -> 2
- net COL0: track 197.6 -> 273.7 mm
- net ROW0: track 228.6 -> 301.0 mm, vias 0 -> 2
- net COL7: track 106.4 -> 168.9 mm
- net COL1: track 109.5 -> 154.2 mm
- net COL2: track 109.4 -> 151.0 mm, vias 0 -> 2
- net COL6: track 104.7 -> 137.7 mm
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