File: 4060.kicad_pcb (KiCad board)
At the start: 2 copper layers, 248 x 99.2 mm, 137 parts, among them J1 JST, SW1 SW_Push, SW10 SW_Push, SW11 SW_Push, SW12 SW_Push, SW13 SW_Push, SW14 SW_Push, SW15 SW_Push, SW16 SW_Push, SW17 SW_Push, SW18 SW_Push, SW19 SW_Push, SW2 SW_Push, SW20 SW_Push, SW21 SW_Push, SW22 SW_Push, SW23 SW_Push, SW24 SW_Push, SW24_1 SW_Push, SW25 SW_Push, SW26 SW_Push, SW27 SW_Push, SW28 SW_Push, SW29 SW_Push, SW3 SW_Push, SW30 SW_Push, SW31 SW_Push, SW32 SW_Push, SW33 SW_Push, SW34 SW_Push, SW35 SW_Push, SW35_1 SW_Push, SW35_2 SW_Push, SW36 SW_Push, SW36_1 SW_Push, SW37 SW_Push, SW38 SW_Push, SW39 SW_Push, SW4 SW_Push, SW40 SW_Push, SW41 SW_Push, SW42 SW_Push, SW43 SW_Push, SW44 SW_Push, SW45 SW_Push, SW46 SW_Push, SW47 SW_Push, SW47_1 SW_Push, SW48 SW_Push, SW48_1 SW_Push, SW49 SW_Push, SW5 SW_Push, SW50 SW_Push, SW51 SW_Push, SW52 SW_Push, SW53 SW_Push, SW54 SW_Push, SW55 SW_Push, SW56 SW_Push, SW56_1 SW_Push, SW57 SW_Push, SW57_1 SW_Push, SW58 RST, SW59 RST, SW6 SW_Push, SW7 SW_Push, SW8 SW_Push, SW9 SW_Push, U1 STM32F072C8Tx, U2 XC6206PxxxMR-Regulator_Linear

Commit message: Routing fixes
Routing:
- net COL4: track 68.7 -> 60.1 mm
- net ROW1: track 290.7 -> 287.7 mm
- net COL5: track 101.7 -> 99.9 mm
- net COL3: track 110.0 -> 108.6 mm
- net COL2: track 134.9 -> 133.5 mm
- net Net-(D48-A): track 28.3 -> 27.5 mm
- net COL10: track 242.8 -> 242.1 mm
- net COL11: track 344.6 -> 343.8 mm
Other:
- board text added: "40/60 Rev. 1"
